File: PCB_iter_3.brd (EAGLE design)
At the start: 100.7 x 58.6 mm, 47 parts, among them IC1 REF5025AID, IC2 REF5025AID, J3 USB_C, P1 M-1X08-SIP-100-40, P2 M-1X08-SIP-100-40, P3 M-1X06-SIP-100-40, P4 M-1X10-SIP-100-40, U2 AD1580, U3 MAX680CPA+, U4 TL072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

Commit message: PCB ITERATION 4
Parts:
- C11, C8, C9, SPARE: device adafruit:C0805 -> adafruit:C1206
- moved R19 20.9 mm to (63.0, 37.6), turned to 180 degrees
- moved R10 11.3 mm to (74.7, 42.6), turned to 270 degrees
- moved C7 8.64 mm to (86.1, 35.3), turned to 90 degrees
- moved C1 7.95 mm to (88.6, 51.1), turned to 180 degrees
- moved R13 7.26 mm to (48.3, 33.2)
- moved U2 5.17 mm to (40.7, 31.9)
- moved C4 4.57 mm to (95.5, 43.7), turned to 270 degrees
- moved R8 3.93 mm to (40.5, 9.65)
- moved C2 3.39 mm to (81.8, 43.4)
- moved R7 3.20 mm to (46.8, 10.9)
- moved C5 2.82 mm to (36.0, 22.3)
- moved C12 2.30 mm to (40.6, 5.99)
- moved U4 2.17 mm to (76.5, 34.0)
- moved C6 1.59 mm to (22.9, 14.6)
- moved R2 0.91 mm to (94.0, 9.10), turned to 180 degrees
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Routing:
- net -12V: track 63.8 -> 43.8 mm
- net OA3_IN-: track 28.1 -> 9.50 mm
- net +12V: track 63.8 -> 45.3 mm
- net ADC_I/P: track 44.2 -> 33.9 mm
- net OA3_IN+: track 116.8 -> 126.6 mm
- net OA1_IN-: track 25.0 -> 33.4 mm
- net +5V: track 203.5 -> 211.4 mm
- net OA4_IN+: track 23.0 -> 29.4 mm
- net N$2: track 14.3 -> 8.08 mm
- net N$5: track 11.8 -> 6.14 mm
- net OA1_IN+: track 15.1 -> 20.1 mm
- net OA1_O/P: track 26.4 -> 31.4 mm
- net N$9: track 3.72 -> 8.25 mm
- net OA2_IN-: track 30.0 -> 34.2 mm
- net N$6: track 25.9 -> 23.0 mm
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